Commit message: clean and fix ns

File: examples/balancer.sdf.xacro (robot description, xacro)
@@ -1,3 +1,3 @@
-<sdf version="1.7" xmlns:xacro="http://dd">
+<sdf version="1.7" xmlns:xacro="http://xacro">
     <xacro:include uri="file://data.xacro" />
     <xacro:include uri="package://common.xacro" />
@@ -9,5 +9,5 @@
         <link name="heavy_base_link">
             <!-- position the base such that the bottom touches the floor -->
-            <pose>0 0 0.55 0 0 0</pose>
+            <pose>0 0 0.55 0 ${PI/2} 0</pose>
             <inertial>
                 <xacro:inertia_box m="${base_mass}" x="${base_x}" y="${base_y}" z="${base_z}" />
@@ -16,12 +16,4 @@
             <collision name="heavy_base_collision">
                 <xacro:geometry_box x="${base_x}" y="${base_y}" z="${base_z}"/>
-                <surface>
-                    <friction>
-                      <ode>
-                        <mu>0</mu>
-                        <mu2>0</mu2>
-                      </ode>
-                    </friction>
-                  </surface>
             </collision>
             <!-- Same geometry as collision -->
@@ -68,4 +60,25 @@
         <xacro:wheel_joint prefix="left" wheel="wheel_left" parent="heavy_base_link"/>
         <xacro:wheel_joint prefix="right" wheel="wheel_right" parent="heavy_base_link"/>
+        <link name="imu_base">
+            <pose relative_to="heavy_base_link">-${(base_x/2)-0.1} 0 0.1 0 0 0</pose>
+            <inertial>
+                <xacro:inertia_box m="0.1" x="0.1" y="0.1" z="0.1"/>
+            </inertial>
+            <!-- Same geometry as visual -->
+            <collision name="imu_base_collision">
+                <xacro:geometry_box x="0.1" y="0.1" z="0.1"/>
+            </collision>
+            <!-- Same geometry as collision -->
+            <visual name="imu_base_visual">
+                <xacro:geometry_box x="0.1" y="0.1" z="0.1"/>
+                <material>
+                    <xacro:color color_name="Black"/>
+                </material>
+            </visual>
+        </link>
+        <joint name="imu_base_joint" type="fixed">
+            <parent>heavy_base_link</parent>
+            <child>imu_base</child>
+          </joint>
     </model>
 </sdf>

File: examples/data.xacro (robot description, xacro)
@@ -1,4 +1,5 @@
-<sdf xmlns:xacro="http://dd">
-    <xacro:property name="base_mass" value="200" />
+<sdf xmlns:xacro="http://xacro">
+    <xacro:property name="PI" value="3.14" />
+    <xacro:property name="base_mass" value="2" />
     <xacro:property name="bodylen" value=".6" />
     <xacro:property name="base_x" value="2.2" />

File: examples/property.xacro (robot description, xacro)
@@ -1,3 +1,3 @@
-<sdf xmlns:xacro="http://dd">
+<sdf xmlns:xacro="http://xacro">
     <xacro:property name="width" value=".2" />
     <xacro:property name="bodylen" value=".6" />
@@ -11,13 +11,5 @@
                 <cylinder radius="${2*width}" length="${bodylen}" />
             </geometry>
-            <material name="blue">
-                <color rgba="0 0 .8 1" />
-            </material>
         </visual>
-        <collision>
-            <geometry>
-                <cylinder radius="${width}" length="${bodylen}" />
-            </geometry>
-        </collision>
     </link>
 </sdf>

File: src/helpers/color.xacro (robot description, xacro)
@@ -1,3 +1,3 @@
-<sdf xmlns:xacro="http://dd">
+<sdf xmlns:xacro="http://xacro">
     <xacro:macro name="color" params="color_name">
         <lighting>1</lighting>

File: src/helpers/common.xacro (robot description, xacro)
@@ -1,4 +1,5 @@
 <?xml version="1.0"?>
-<sdf xmlns:xacro="http://dd">
+<sdf xmlns:xacro="http://xacro">
+<!-- inertia_box -->
 <xacro:macro name="inertia_box" params="m x y z">
     <mass>${m}</mass>
@@ -10,4 +11,16 @@
         <iyz>0</iyz>
         <izz>${m*(x*x+y*y)/12}</izz>
+    </inertia>
+</xacro:macro>
+<!-- inertia_sphere -->
+<xacro:macro name="inertia_sphere" params="m r">
+    <mass>${m}</mass>
+    <inertia>
+        <ixx>${2*m*r*r/5}</ixx>
+        <ixy>0</ixy>
+        <ixz>0</ixz>
+        <iyy>${2*m*r*r/5}</iyy>
+        <iyz>0</iyz>
+        <izz>${2*m*r*r/5}</izz>
     </inertia>
 </xacro:macro>
@@ -41,3 +54,11 @@
     </geometry>
 </xacro:macro>
+<!-- geometry_sphere -->
+<xacro:macro name="geometry_sphere" params="r">
+    <geometry>
+        <sphere>
+            <radius>${r}</radius>
+        </sphere>
+    </geometry>
+</xacro:macro>
 </sdf>

Commit message: sdf exemples

File: examples/balancer.sdf.xacro (robot description, xacro)
@@ -83,4 +83,5 @@
             <child>imu_base</child>
           </joint>
+          <plugin name="simple_plug" filename="libsimple_sub.so"/>
     </model>
 </sdf>

File: src/helpers/color.xacro (robot description, xacro)
@@ -1,3 +1,4 @@
 <sdf xmlns:xacro="http://xacro">
+    <!-- color -->
     <xacro:macro name="color" params="color_name">
         <lighting>1</lighting>
@@ -7,3 +8,11 @@
         </script>
     </xacro:macro>
+    <!-- texture -->
+    <xacro:macro name="texture" params="model name">
+        <script>
+            <uri>model://${model}/materials/scripts</uri>
+            <uri>model://${model}/materials/textures</uri>
+            <name>${model}/${name}</name>
+        </script>
+    </xacro:macro>
 </sdf>

File: src/helpers/common.xacro (robot description, xacro)
@@ -1,64 +1,76 @@
 <?xml version="1.0"?>
 <sdf xmlns:xacro="http://xacro">
-<!-- inertia_box -->
-<xacro:macro name="inertia_box" params="m x y z">
-    <mass>${m}</mass>
-    <inertia>
-        <ixx>${m*(y*y+z*z)/12}</ixx>
-        <ixy>0</ixy>
-        <ixz>0</ixz>
-        <iyy>${m*(x*x+z*z)/12}</iyy>
-        <iyz>0</iyz>
-        <izz>${m*(x*x+y*y)/12}</izz>
-    </inertia>
-</xacro:macro>
-<!-- inertia_sphere -->
-<xacro:macro name="inertia_sphere" params="m r">
-    <mass>${m}</mass>
-    <inertia>
-        <ixx>${2*m*r*r/5}</ixx>
-        <ixy>0</ixy>
-        <ixz>0</ixz>
-        <iyy>${2*m*r*r/5}</iyy>
-        <iyz>0</iyz>
-        <izz>${2*m*r*r/5}</izz>
-    </inertia>
-</xacro:macro>
-<!-- inertia_cylinder -->
-<xacro:macro name="inertia_cylinder" params="m r l">
-    <mass>${m}</mass>
-    <inertia>
-        <ixx>${m*(3*r*r+l*l)/12}</ixx>
-        <ixy>0</ixy>
-        <ixz>0</ixz>
-        <iyy>${m*(3*r*r+l*l)/12}</iyy>
-        <iyz>0</iyz>
-        <izz>${m*r*r/2}</izz>
-    </inertia>
-</xacro:macro>
-<!-- geometry_cylinder -->
-<xacro:macro name="geometry_cylinder" params="r l">
-    <geometry>
-        <cylinder>
-            <radius>${r}</radius>
-            <length>${l}</length>
-        </cylinder>
-    </geometry>
-</xacro:macro>
-<!-- geometry_box -->
-<xacro:macro name="geometry_box" params="x y z">
-    <geometry>
-        <box>
-            <size>${x} ${y} ${z}</size>
-        </box>
-    </geometry>
-</xacro:macro>
-<!-- geometry_sphere -->
-<xacro:macro name="geometry_sphere" params="r">
-    <geometry>
-        <sphere>
-            <radius>${r}</radius>
-        </sphere>
-    </geometry>
-</xacro:macro>
+    <!-- inertia_box -->
+    <xacro:macro name="inertia_box" params="m x y z">
+        <mass>${m}</mass>
+        <inertia>
+            <ixx>${m*(y*y+z*z)/12}</ixx>
+            <ixy>0</ixy>
+            <ixz>0</ixz>
+            <iyy>${m*(x*x+z*z)/12}</iyy>
+            <iyz>0</iyz>
+            <izz>${m*(x*x+y*y)/12}</izz>
+        </inertia>
+    </xacro:macro>
+    <!-- inertia_sphere -->
+    <xacro:macro name="inertia_sphere" params="m r">
+        <mass>${m}</mass>
+        <inertia>
+            <ixx>${2*m*r*r/5}</ixx>
+            <ixy>0</ixy>
+            <ixz>0</ixz>
+            <iyy>${2*m*r*r/5}</iyy>
+            <iyz>0</iyz>
+            <izz>${2*m*r*r/5}</izz>
+        </inertia>
+    </xacro:macro>
+    <!-- inertia_cylinder -->
+    <xacro:macro name="inertia_cylinder" params="m r l">
+        <mass>${m}</mass>
+        <inertia>
+            <ixx>${m*(3*r*r+l*l)/12}</ixx>
+            <ixy>0</ixy>
+            <ixz>0</ixz>
+            <iyy>${m*(3*r*r+l*l)/12}</iyy>
+            <iyz>0</iyz>
+            <izz>${m*r*r/2}</izz>
+        </inertia>
+    </xacro:macro>
+    <!-- geometry_cylinder -->
+    <xacro:macro name="geometry_cylinder" params="r l">
+        <geometry>
+            <cylinder>
+                <radius>${r}</radius>
+                <length>${l}</length>
+            </cylinder>
+        </geometry>
+    </xacro:macro>
+    <!-- geometry_box -->
+    <xacro:macro name="geometry_box" params="x y z">
+        <geometry>
+            <box>
+                <size>${x} ${y} ${z}</size>
+            </box>
+        </geometry>
+    </xacro:macro>
+    <!-- geometry_sphere -->
+    <xacro:macro name="geometry_sphere" params="r">
+        <geometry>
+            <sphere>
+                <radius>${r}</radius>
+            </sphere>
+        </geometry>
+    </xacro:macro>
+    <xacro:macro name="box_vc" params="name x y z color">
+        <collision name="${name}_collision">
+            <xacro:geometry_box x="${x}" y="${y}" z="${z}" />
+        </collision>
+        <!-- Same geometry as collision -->
+        <visual name="${name}_visual">
+            <xacro:geometry_box x="${x}" y="${y}" z="${z}" />
+            <material>
+                <xacro:color color_name="${color}" />
+            </material>
+        </visual>
+    </xacro:macro>
 </sdf>

File: src/helpers/sensors.xacro (robot description, xacro)
@@ -1,12 +1,37 @@
 <?xml version="1.0"?>
 <sdf xmlns:xacro="http://xacro">
-<!-- __default_topic__ -->
-<xacro:macro name="imu" params="name rate topic">
-    <sensor name="${name}" type="imu">
-        <always_on>true</always_on>
-        <update_rate>${rate}</update_rate>
-        <visualize>true</visualize>
-        <topic>${topic}</topic>
-    </sensor>
-</xacro:macro>
+    <!-- IMU -->
+    <xacro:macro name="imu" params="name rate topic">
+        <sensor name="${name}" type="imu">
+            <always_on>true</always_on>
+            <update_rate>${rate}</update_rate>
+            <visualize>true</visualize>
+            <topic>${topic}</topic>
+        </sensor>
+    </xacro:macro>
+    <!-- camera -->
+    <xacro:macro name="camera" params="name rate width height fov">
+        <sensor type="camera" name="${name}">
+            <update_rate>${rate}</update_rate>
+            <visualize>1</visualize>
+            <!-- <pose>0.025 0 0 0 0 0</pose> -->
+            <camera name="head">
+                <horizontal_fov>${fov*PI/180}</horizontal_fov>
+                <image>
+                    <width>${width}</width>
+                    <height>${height}</height>
+                    <format>R8G8B8</format>
+                </image>
+                <clip>
+                    <near>0.02</near>
+                    <far>300</far>
+                </clip>
+                <noise>
+                    <type>gaussian</type>
+                    <mean>0.0</mean>
+                    <stddev>0.007</stddev>
+                </noise>
+            </camera>
+        </sensor>
+    </xacro:macro>
 </sdf>
